Commit message: feat: reference gait, MATLAB player, and measured motor mass
Two changes that belong together: a walking reference gait for the published
URDF (with a MATLAB player and preview media), and a motor-mass correction that
brings the model in line with a measurement.

Reference gait and MATLAB player
- tools/matlab/wamoduck_play.m: interactive player. Play/pause, advance step,
  switch between two data sets, skeleton or full-mesh view, a torque plot
  against the motor's rated and peak values, and a per-joint table.
- tools/matlab/data/: one steady-state gait cycle (2.0 s, 100 frames at 50 Hz,
  loops seamlessly) and the full 1 m walk decimated to 10 Hz. Joint angles in
  radians and inverse-dynamics torque estimates in N*m, so nothing in the
  replay path needs a unit conversion.
- assets/: a two-cycle GIF, a 20 s walk video, a still frame, and a screenshot
  of the player. Rendered from the public URDF by prescribing the joint angles
  and running forward kinematics; no physics integration, no controller.
- docs/matlab.en.md and docs/matlab.zh-CN.md: data format, scope, and the
  measured limits of this leg design. There is no ankle-roll joint, and a
  single-support step would need at least 57 mm of lateral centre-of-mass
  travel, so the plan is a double-support quasi-static shuffle with a 4.5 mm
  foot lift.
- Readme section in both languages, plus assets/README.md, media-manifest.json
  entries with per-asset scope notes, and .gitattributes/.gitignore updates.

Motor mass
- wmduck.urdf: the 15 motor instances now use the measured 141 g instead of the
  150 g transcribed from the vendor parameter image. Model total mass
  3.886339783 -> 3.751339783 kg. Motor centres of mass stay at their CAD
  positions and motor inertias are rescaled by mass ratio, so every link that
  carries a motor changed slightly in mass, centre of mass, and inertia.
  Geometry, joint definitions, and the zero-pose envelope are unchanged.
- motor_parameters.json: records the basis and date of the mass value, lists
  the 3.6 N*m peak alongside the 3.7 N*m stall figure, and records a bench
  observation that the motor held 3.5 N*m for more than 30 s. That observation
  is labelled as one observation, not a duty-cycle or thermal rating, and the
  rated 0.6 N*m is unchanged.
- component_mass_audit.csv and validation.json regenerated: the audit mass
  column sums to the URDF model mass to within 1e-9 kg, and validation.json
  keeps the previous values under revision_note.
- READMEs and docs/model.*: mass figures and the motor-data narrative updated.
- asset-manifest.json and media-manifest.json carry the new hashes, and the
  URDF transformation note no longer claims "model numerical data unchanged".

Verification
- Gait data, via the player's self-test: all 15 joints inside the URDF limits,
  and both soles within 0.1 mm of the ground plane by URDF forward kinematics,
  agreeing with the model-side measurement.
- The shipped cycle is a steady-state cycle (same-phase frames of consecutive
  cycles agree to 0.000 degrees) and its loop seam equals one frame step
  (0.13 degrees).
- After the mass update, per-link mass/centre-of-mass/inertia changes are
  confined to links that carry a motor, and the zero-pose envelope is
  unchanged. The sum of component_mass_audit.csv equals the URDF model mass.
- Text data is stored LF-normalized, so the SHA-256 values recorded in the
  media manifest match the bytes as committed (this repository sets
  `* text=auto eol=lf`).

Scope: the gait is a kinematic inverse-kinematics plan with a static-stability
check. It is not a trained policy, not hardware data, and not a dynamic-balance
result. The motor mass and the 30 s torque observation are maintainer
measurements; other component masses remain CAD values.

File: models/wmduck/wmduck.urdf (robot description, URDF)
Before this commit: robot wmduck, 17 links, 16 joints
Links:
- link base_link: mass 0.66864023518 -> 0.65064023518
- link head_roll_link: mass 1.09884048193 -> 1.08084048193
- link head_yaw_link: mass 0.160466330426 -> 0.151466330426
- link left_ankle_link: mass 0.225671675043 -> 0.216671675043
- link left_hip_pitch_link: mass 0.327377727974 -> 0.309377727974
- link left_hip_yaw_link: mass 0.160466330426 -> 0.151466330426
- link neck_pitch_link: mass 0.345409232363 -> 0.327409232363
- link right_ankle_link: mass 0.225671675042 -> 0.216671675042
- link right_hip_pitch_link: mass 0.327377727974 -> 0.309377727974
- link right_hip_yaw_link: mass 0.160466330426 -> 0.151466330426
